Commit message: WT-600 차체 확정 반영: WHEEL_BASE 0.190→0.245(실측), URDF 전면 개정, S2L/D455f 마운트

File: Docs/rover.urdf (robot description, URDF)
Before this commit: robot jupiter_rover, 8 links, 7 joints
Links:
- removed link battery_link
- removed link computing_board_link
- added link imu_link
- added link sensor_deck_link; visual box size=0.178 0.132 0.005; visual cylinder length=0.084 radius=0.0085
- link base_link: mass 3.0 -> 8.5; geometry collision box size=0.50 0.25 0.105; visual box size=0.50 0.25 0.105
- link camera_link: geometry visual box size=0.026 0.124 0.029
- link left_track: mass None -> 0.6; geometry collision box size=0.50 0.04 0.105; visual box size=0.50 0.04 0.105
- link lidar_link: geometry visual cylinder length=0.0398 radius=0.0385
- link right_track: mass None -> 0.6; geometry collision box size=0.50 0.04 0.105; visual box size=0.50 0.04 0.105
Joints:
- removed joint battery_joint
- removed joint computing_board_joint
- added joint imu_joint: type fixed, parent base_link, child imu_link, origin xyz=0 0 0.09 rpy=0 -0.0611 0
- added joint sensor_deck_joint: type fixed, parent base_link, child sensor_deck_link, origin xyz=0.152 0.0 0.159 rpy=0 0 0
- joint base_joint: origin xyz=0 0 0.025 rpy=0 0 0 -> xyz=0 0 0.02567 rpy=0 0 0
- joint camera_joint: origin xyz=0.13 0.0 0.08 rpy=0 0 0 -> xyz=0.232 0.0475 0.143 rpy=0 0 0
- joint left_track_joint: origin xyz=0 0.095 0 rpy=0 0 0 -> xyz=0 0.1225 0.027 rpy=0 0 0
- joint lidar_joint: origin xyz=0.02 0.0 0.12 rpy=0 0 0 -> xyz=0.152 0.0 0.185 rpy=0 0 0
- joint right_track_joint: origin xyz=0 -0.095 0 rpy=0 0 0 -> xyz=0 -0.1225 0.027 rpy=0 0 0
