Commit message: 09-18 §9 센서 데크 yaw −2.68° 보정: 로컬 코스트맵 상자 드리프트의 원인. 라이다 yaw π→3.09482, 카메라 yaw −0.04677·위치 회전, stuck_monitor 동기화
- bag(mp9~12): SLAM 옆 보정이 회전 방향과 무관하게 항상 왼쪽 +4 cm/m, 게걸음 각 +2.69°(곡률·heading 무관) → 옆미끄럼 가설 기각, 장착 yaw 오차 모양
- 정지 측정(오른쪽 옆면을 벽에 접촉): 라이다 +2.667/+2.686°, 카메라 +2.94°(같은 벽) → 데크 전체 회전. 동적·정적 0.03° 일치
- 보정 후 TF 기준 같은 벽 −0.031° 확인. Jetson 배포(백업 ~/ros2_ws/.bak_20260918)
- 주행 판정 기준 선언: 게걸음 각 |평균|<0.7°, 옆 보정 <2 cm/주행, 로컬−전역 상자 차 <2 cm

Co-Authored-By: Claude Opus 5 (1M context) <noreply@anthropic.com>

File: Docs/rover.urdf (robot description, URDF)
Before this commit: robot jupiter_rover, 8 links, 7 joints
Joints:
- joint camera_joint: origin xyz=0.232 0.0475 0.143 rpy=0 0 0 -> xyz=0.23413 0.04371 0.143 rpy=0 0 -0.04677
- joint lidar_joint: origin xyz=0.152 0.0 0.185 rpy=0 0 3.14159265 -> xyz=0.152 0.0 0.185 rpy=0 0 3.09482
- joint sensor_deck_joint: origin xyz=0.152 0.0 0.159 rpy=0 0 0 -> xyz=0.152 0.0 0.159 rpy=0 0 -0.04677

File: ros2_ws/src/rover_description/urdf/rover.urdf.xacro (robot description, xacro)
@@ -12,4 +12,6 @@
   <xacro:arg name="deck_y"        default="0.000"/>
   <xacro:arg name="lidar_yaw"     default="3.14159265"/>
+  <!-- 2026-09-18 데크 yaw 실측 −2.68° (rover.urdf 확정본과 같은 값): 라이다·카메라가 함께 회전, 카메라 위치는 데크 원점 기준 회전 -->
+  <xacro:arg name="deck_yaw"      default="-0.04677"/>
   <xacro:property name="base_z"      value="0.025"/>
   <xacro:property name="deck_t"      value="0.005"/>
@@ -24,4 +26,5 @@
   <xacro:property name="cam_dy"      value="0.0475"/>
   <xacro:property name="cam_dz"      value="-0.0165"/>
+  <xacro:property name="deck_yaw"    value="$(arg deck_yaw)"/>
   <material name="green"><color rgba="0.1 0.7 0.3 1.0"/></material>
   <material name="black"><color rgba="0.1 0.1 0.1 1.0"/></material>
@@ -53,5 +56,5 @@
     <!-- 센서 데크 (FUSED_ROVER STL, mm → m), 데크 프레임 원점에 배치 -->
     <visual>
-      <origin xyz="${deck_x} ${deck_y} ${deck_bottom - base_z}" rpy="0 0 0"/>
+      <origin xyz="${deck_x} ${deck_y} ${deck_bottom - base_z}" rpy="0 0 ${deck_yaw}"/>
       <geometry><mesh filename="package://rover_description/meshes/sensor_deck.stl" scale="0.001 0.001 0.001"/></geometry>
       <material name="petg"/>
@@ -84,5 +87,5 @@
   <joint name="lidar_joint" type="fixed">
     <parent link="base_link"/><child link="lidar_link"/>
-    <origin xyz="${deck_x} ${deck_y} ${deck_bottom - base_z + lidar_dz}" rpy="0 0 $(arg lidar_yaw)"/>
+    <origin xyz="${deck_x} ${deck_y} ${deck_bottom - base_z + lidar_dz}" rpy="0 0 ${$(arg lidar_yaw) + deck_yaw}"/>
   </joint>
   <!-- ===== RealSense D455f — camera_link = 좌이미저 (드라이버가 하위 optical/imu 프레임 발행) ===== -->
@@ -96,5 +99,5 @@
   <joint name="camera_joint" type="fixed">
     <parent link="base_link"/><child link="camera_link"/>
-    <origin xyz="${deck_x + cam_dx} ${deck_y + cam_dy} ${deck_bottom - base_z + cam_dz}" rpy="0 0 0"/>
+    <origin xyz="${deck_x + cam_dx*cos(deck_yaw) - cam_dy*sin(deck_yaw)} ${deck_y + cam_dx*sin(deck_yaw) + cam_dy*cos(deck_yaw)} ${deck_bottom - base_z + cam_dz}" rpy="0 0 ${deck_yaw}"/>
   </joint>
   <!-- 보드 IMU 프레임 (펌웨어 /imu/data_raw frame_id) — 자이로 무반응 판정으로 미융합, TF 존재만 유지 -->
