Commit message: rover.urdf.xacro 를 확정본 rover.urdf 와 같은 TF 로 재작성(08-27 초안 값 잔존 — 라이다 x 15 cm · z 10 cm 어긋남) · 관절 비교 도구 · stuck_monitor 자이로 우선은 켜지 않음(사용자)
Co-Authored-By: Claude Opus 5.5 <noreply@anthropic.com>
Claude-Session: https://claude.ai/code/session_01KWQmAZCE2vxYuVEwKt2nZZ

File: ros2_ws/src/rover_description/urdf/rover.urdf.xacro (robot description, xacro)
@@ -1,33 +1,31 @@
 <?xml version="1.0" ?>
-<!-- Jupiter rover URDF (xacro) — 센서 데크(FUSED_ROVER) 반영판. 2026-08-27
-     좌표: ROS(X전방/Y좌/Z상). base_footprint = 지면, base_link = +0.025 (휠 유효반경 0.02567 근사)
-     데크 프레임: 원점 = LiDAR 마운트 중심·데크 하면 (gen_rover_deck.py 기준)
-     장착 후 실측 인자 (TODO: 측정 전까지 기본값은 추정치):
-       lidar_mount_h : 지면 → LiDAR 하면(=데크 상면) 높이 [m]
-       deck_x, deck_y: LiDAR 마운트 중심의 base_link 기준 전후/좌우 오프셋 [m] (트랙 길이 중점 기준)
-       lidar_yaw     : rplidar_ros x축이 하드웨어 후방을 향하므로 보통 π (h_axis_check 절차로 실측 확정) -->
+<!-- Jupiter rover URDF (xacro) — 확정본 rover.urdf 와 같은 TF 트리 · 같은 값 + 데크 인자화 · 데크 메시 시각화.
+     2026-10-30 재작성: 이전 판(08-27 초안)은 WT-600 개정 전 값(데크 x 0 · 카메라 dx 0.0822 · 트랙 y ±0.095 ·
+     base_z 0.025 · sensor_deck_link 없음)이 남아 있어 use_xacro:=true 로 띄우면 라이다 · 카메라가 x 로 약 15 cm 어긋났다
+     (Docs/issues/sensor-deck-yaw.md). 값의 근거는 rover.urdf 주석 — 여기서는 그 값을 기본으로 쓴다.
+     좌표: ROS(X전방/Y좌/Z상). base_footprint = 지면, base_link = +0.02567(휠 유효 구름 반경).
+     인자(기본 = rover.urdf 확정값; 데크를 다시 조립하면 재측정 — CLAUDE.md 하드웨어 요약 ⚠):
+       deck_x, deck_y : 데크 원점(라이다 마운트 중심, 판 하면) 의 base_link 기준 위치 [m]
+       deck_z         : 같은 원점의 높이 [m] (= 판 하면 지면高 0.185 − 0.02567)
+       deck_yaw       : 데크 장착 yaw [rad] (2026-09-18 실측 −2.68°)
+       lidar_yaw      : 데크 기준 라이다 yaw [rad] (π — RPLidar 하드웨어 0° = 로버 후방, 2026-08-28) -->
 <robot name="jupiter_rover" xmlns:xacro="http://www.ros.org/wiki/xacro">
-  <xacro:arg name="lidar_mount_h" default="0.290"/>
-  <xacro:arg name="deck_x"        default="0.000"/>
-  <xacro:arg name="deck_y"        default="0.000"/>
-  <xacro:arg name="lidar_yaw"     default="3.14159265"/>
-  <!-- 2026-09-18 데크 yaw 실측 −2.68° (rover.urdf 확정본과 같은 값): 라이다·카메라가 함께 회전, 카메라 위치는 데크 원점 기준 회전 -->
-  <xacro:arg name="deck_yaw"      default="-0.04677"/>
-  <xacro:property name="base_z"      value="0.025"/>
-  <xacro:property name="deck_t"      value="0.005"/>
-  <xacro:property name="scan_above"  value="0.0208"/>
-  <xacro:property name="lidar_mount_h" value="$(arg lidar_mount_h)"/>
-  <xacro:property name="deck_bottom" value="${lidar_mount_h - deck_t}"/>
-  <xacro:property name="deck_x"      value="$(arg deck_x)"/>
-  <xacro:property name="deck_y"      value="$(arg deck_y)"/>
-  <!-- 데크 원점 기준 센서 오프셋 (CAD + Intel xacro 확정값) -->
-  <xacro:property name="lidar_dz"    value="${deck_t + scan_above}"/>
-  <xacro:property name="cam_dx"      value="0.0822"/>
-  <xacro:property name="cam_dy"      value="0.0475"/>
-  <xacro:property name="cam_dz"      value="-0.0165"/>
-  <xacro:property name="deck_yaw"    value="$(arg deck_yaw)"/>
+  <xacro:arg name="deck_x"    default="0.152"/>
+  <xacro:arg name="deck_y"    default="0.0"/>
+  <xacro:arg name="deck_z"    default="0.159"/>
+  <xacro:arg name="deck_yaw"  default="-0.04677"/>
+  <xacro:arg name="lidar_yaw" default="3.14159265"/>
+  <xacro:property name="base_z"   value="0.02567"/>
+  <xacro:property name="deck_x"   value="$(arg deck_x)"/>
+  <xacro:property name="deck_y"   value="$(arg deck_y)"/>
+  <xacro:property name="deck_z"   value="$(arg deck_z)"/>
+  <xacro:property name="deck_yaw" value="$(arg deck_yaw)"/>
+  <!-- 데크 원점 기준 센서 오프셋 (rover.urdf 확정값: 라이다 z 0.185 − 0.159, 카메라 (0.080, 0.0475, 0.143 − 0.159)) -->
+  <xacro:property name="lidar_dz" value="0.026"/>
+  <xacro:property name="cam_dx"   value="0.080"/>
+  <xacro:property name="cam_dy"   value="0.0475"/>
+  <xacro:property name="cam_dz"   value="-0.016"/>
   <material name="green"><color rgba="0.1 0.7 0.3 1.0"/></material>
   <material name="black"><color rgba="0.1 0.1 0.1 1.0"/></material>
-  <material name="blue"><color rgba="0.1 0.3 0.9 1.0"/></material>
   <material name="grey"><color rgba="0.6 0.6 0.6 1.0"/></material>
   <material name="dark_grey"><color rgba="0.3 0.3 0.3 1.0"/></material>
@@ -39,46 +37,60 @@
     <origin xyz="0 0 ${base_z}" rpy="0 0 0"/>
   </joint>
+  <!-- 차체: WT-600 본체 (트랙 제외 폭 0.25) -->
   <link name="base_link">
     <visual>
-      <origin xyz="0 0 0.03" rpy="0 0 0"/>
-      <geometry><box size="0.24 0.14 0.06"/></geometry>
+      <origin xyz="0 0 0.027" rpy="0 0 0"/>
+      <geometry><box size="0.50 0.25 0.105"/></geometry>
       <material name="green"/>
     </visual>
     <collision>
-      <origin xyz="0 0 0.03" rpy="0 0 0"/>
-      <geometry><box size="0.24 0.14 0.06"/></geometry>
+      <origin xyz="0 0 0.027" rpy="0 0 0"/>
+      <geometry><box size="0.50 0.25 0.105"/></geometry>
     </collision>
     <inertial>
-      <mass value="3.0"/>
+      <mass value="8.5"/>
+      <origin xyz="0 0 0.027" rpy="0 0 0"/>
+      <inertia ixx="0.0521" ixy="0.0" ixz="0.0" iyy="0.1849" iyz="0.0" izz="0.2214"/>
+    </inertial>
+  </link>
+  <xacro:macro name="track" params="side y">
+    <link name="${side}_track">
+      <visual><origin xyz="0 0 0" rpy="0 0 0"/><geometry><box size="0.50 0.04 0.105"/></geometry><material name="black"/></visual>
+      <collision><origin xyz="0 0 0" rpy="0 0 0"/><geometry><box size="0.50 0.04 0.105"/></geometry></collision>
+      <inertial>
+        <mass value="0.6"/>
+        <origin xyz="0 0 0" rpy="0 0 0"/>
+        <inertia ixx="0.00063" ixy="0.0" ixz="0.0" iyy="0.01305" iyz="0.0" izz="0.01258"/>
+      </inertial>
+    </link>
+    <joint name="${side}_track_joint" type="continuous">
+      <parent link="base_link"/><child link="${side}_track"/>
+      <origin xyz="0 ${y} 0.027" rpy="0 0 0"/><axis xyz="0 1 0"/>
+    </joint>
+  </xacro:macro>
+  <xacro:track side="left"  y="0.1225"/>
+  <xacro:track side="right" y="-0.1225"/>
+  <!-- 보드 IMU (ICM-20948, 상판 3.5° 기울기 상속) — 자이로 무반응으로 미융합, TF 만 유지 -->
+  <link name="imu_link"/>
+  <joint name="imu_joint" type="fixed">
+    <parent link="base_link"/><child link="imu_link"/>
+    <origin xyz="0 0 0.09" rpy="0 -0.0611 0"/>
+  </joint>
+  <!-- 센서 데크: 원점 = 라이다 마운트 중심 · 판 하면. 시각화 = FUSED_ROVER 메시(mm → m, 같은 원점) -->
+  <link name="sensor_deck_link">
+    <visual>
       <origin xyz="0 0 0" rpy="0 0 0"/>
-      <inertia ixx="0.01" ixy="0.0" ixz="0.0" iyy="0.01" iyz="0.0" izz="0.01"/>
-    </inertial>
-    <!-- 센서 데크 (FUSED_ROVER STL, mm → m), 데크 프레임 원점에 배치 -->
-    <visual>
-      <origin xyz="${deck_x} ${deck_y} ${deck_bottom - base_z}" rpy="0 0 ${deck_yaw}"/>
       <geometry><mesh filename="package://rover_description/meshes/sensor_deck.stl" scale="0.001 0.001 0.001"/></geometry>
       <material name="petg"/>
     </visual>
   </link>
-  <link name="left_track">
-    <visual><origin xyz="0 0 0" rpy="0 0 0"/><geometry><box size="0.29 0.05 0.055"/></geometry><material name="black"/></visual>
-    <collision><origin xyz="0 0 0" rpy="0 0 0"/><geometry><box size="0.29 0.05 0.055"/></geometry></collision>
-  </link>
-  <joint name="left_track_joint" type="continuous">
-    <parent link="base_link"/><child link="left_track"/>
-    <origin xyz="0 0.095 0" rpy="0 0 0"/><axis xyz="0 1 0"/>
+  <joint name="sensor_deck_joint" type="fixed">
+    <parent link="base_link"/><child link="sensor_deck_link"/>
+    <origin xyz="${deck_x} ${deck_y} ${deck_z}" rpy="0 0 ${deck_yaw}"/>
   </joint>
-  <link name="right_track">
-    <visual><origin xyz="0 0 0" rpy="0 0 0"/><geometry><box size="0.29 0.05 0.055"/></geometry><material name="black"/></visual>
-    <collision><origin xyz="0 0 0" rpy="0 0 0"/><geometry><box size="0.29 0.05 0.055"/></geometry></collision>
-  </link>
-  <joint name="right_track_joint" type="continuous">
-    <parent link="base_link"/><child link="right_track"/>
-    <origin xyz="0 -0.095 0" rpy="0 0 0"/><axis xyz="0 1 0"/>
-  </joint>
-  <!-- ===== LiDAR (RPLidar S2L) — 스캔면 중심 ===== -->
+  <!-- 라이다 RPLidar S2L — lidar_link 원점 = 스캔면 중심. 방향 = 라이다 yaw + 데크 yaw (stuck_monitor.py LIDAR_YAW 와 한 쌍) -->
   <link name="lidar_link">
     <visual>
-      <origin xyz="0 0 ${-scan_above + 0.0199}" rpy="0 0 0"/>
+      <origin xyz="0 0 0" rpy="0 0 0"/>
       <geometry><cylinder radius="0.0385" length="0.0398"/></geometry>
       <material name="black"/>
@@ -87,10 +99,10 @@
   <joint name="lidar_joint" type="fixed">
     <parent link="base_link"/><child link="lidar_link"/>
-    <origin xyz="${deck_x} ${deck_y} ${deck_bottom - base_z + lidar_dz}" rpy="0 0 ${$(arg lidar_yaw) + deck_yaw}"/>
+    <origin xyz="${deck_x} ${deck_y} ${deck_z + lidar_dz}" rpy="0 0 ${$(arg lidar_yaw) + deck_yaw}"/>
   </joint>
-  <!-- ===== RealSense D455f — camera_link = 좌이미저 (드라이버가 하위 optical/imu 프레임 발행) ===== -->
+  <!-- 카메라 RealSense D455f — camera_link = 좌IR이미저. 위치 = 데크 원점 + 데크 yaw 로 돌린 (cam_dx, cam_dy) -->
   <link name="camera_link">
     <visual>
-      <origin xyz="-0.0112 -0.0475 0" rpy="0 0 0"/>
+      <origin xyz="-0.003 -0.0475 0" rpy="0 0 0"/>
       <geometry><box size="0.026 0.124 0.029"/></geometry>
       <material name="grey"/>
@@ -99,25 +111,5 @@
   <joint name="camera_joint" type="fixed">
     <parent link="base_link"/><child link="camera_link"/>
-    <origin xyz="${deck_x + cam_dx*cos(deck_yaw) - cam_dy*sin(deck_yaw)} ${deck_y + cam_dx*sin(deck_yaw) + cam_dy*cos(deck_yaw)} ${deck_bottom - base_z + cam_dz}" rpy="0 0 ${deck_yaw}"/>
-  </joint>
-  <!-- 보드 IMU 프레임 (펌웨어 /imu/data_raw frame_id) — 자이로 무반응 판정으로 미융합, TF 존재만 유지 -->
-  <link name="imu_link"/>
-  <joint name="imu_joint" type="fixed">
-    <parent link="base_link"/><child link="imu_link"/>
-    <origin xyz="-0.01 0.01 0.08" rpy="0 0 0"/>
-  </joint>
-  <link name="battery_link">
-    <visual><origin xyz="0 0 0" rpy="0 0 0"/><geometry><box size="0.12 0.04 0.05"/></geometry><material name="blue"/></visual>
-  </link>
-  <joint name="battery_joint" type="fixed">
-    <parent link="base_link"/><child link="battery_link"/>
-    <origin xyz="-0.06 -0.07 0.04" rpy="0 0 0"/>
-  </joint>
-  <link name="computing_board_link">
-    <visual><origin xyz="0 0 0" rpy="0 0 0"/><geometry><box size="0.10 0.10 0.03"/></geometry><material name="dark_grey"/></visual>
-  </link>
-  <joint name="computing_board_joint" type="fixed">
-    <parent link="base_link"/><child link="computing_board_link"/>
-    <origin xyz="-0.01 0.01 0.06" rpy="0 0 0"/>
+    <origin xyz="${deck_x + cam_dx*cos(deck_yaw) - cam_dy*sin(deck_yaw)} ${deck_y + cam_dx*sin(deck_yaw) + cam_dy*cos(deck_yaw)} ${deck_z + cam_dz}" rpy="0 0 ${deck_yaw}"/>
   </joint>
 </robot>
